Commit message: feat: unify MORLA coordinate and robot runtime contracts
Add shared SO(3)/SE(3) coordinate contracts and Profile-derived solver/tool frames, then inject them through Astral and Nero bringup and teleoperation. Keep Nero's active IK/control target on link7 while retaining the separately named SDK flange measurement interface.

Integrate Profile-scoped joint-state to TF assembly, kinematics identity in data and policy paths, XNero import compatibility, and the Web profile status changes. Restore the legacy Nero J2 model as an explicitly versioned asset and add Astral/Nero coordinate, state bridge, and simulation integration regressions.

Validation: symlink build 31/31; Profile validation 12/12; coordinate and flange-topic tests 8 passed; Nero FK audit 501 poses per side; VR-to-link7 regression 8/8; git diff --check passed.

File: src/robot_description/urdf/nero/xhand_nero_description.urdf (robot description, URDF)
Before this commit: robot xhand_nero, 1282 links, 1281 joints
Joints:
- joint left_joint2: limit lower=-3.3108 upper=0.1692 effort=100 velocity=5 -> lower=-1.74533 upper=1.74533 effort=100 velocity=5; origin xyz=0 0 0 rpy=0 1.5708 -1.5708 -> xyz=0 0 0 rpy=1.5707963 3.1415926 0
- joint right_joint2: limit lower=-3.3108 upper=0.1692 effort=100 velocity=5 -> lower=-1.74533 upper=1.74533 effort=100 velocity=5; origin xyz=0 0 0 rpy=0 1.5708 -1.5708 -> xyz=0 0 0 rpy=1.5707963 3.1415926 0

Commit message: feat: 集成钢琴工作台并完善 Nero/XHand 控制链路
依据 2026-10-20—22 CHANGELOG、钢琴调试日志及现有工作区保存集成基线。

- 接入独立 MORLA-piano，引入专用 worker、设备互斥、浏览器/进程心跳及会话快照。
- 提供曲谱管理、预检、在线关节/笛卡尔标定、工作位、直接重播及服务端演奏进度。
- 完善 Nero 使能与反馈确认、HOME/工作位轨迹、连续保持目标及钢琴专用 J7/J 模式。
- 同步 XHAND 1 限位、左右手串口关联、被动反馈初始化与原生 SDK 诊断。
- 保存操作输入路由、语音/脚踏、Quest 预览与断流处理、采集确认/QoS及相机配置改动。
- 收录手册、配置归档、部署哈希、SDK误写事件和异机恢复说明，保留历史验收边界。
- 更新前端源码与生产资源，修正 pnpm esbuild 构建配置，排除依赖缓存和运行数据。

配套 MORLA-piano: 1dcd032665cfa2876ab92667fb0ff3e0c3dc4f3c

本次验证：
- 外部引擎 unittest：26 通过；前端 node 测试：18 通过。
- pnpm frozen-lockfile 安装、TypeScript/Vite 生产构建通过。
- 新增/修改 Python 源码 97 个通过语法解析；git diff --cached --check 通过。
- macOS Python 3.9 定向回归：171 通过、6 失败、1 跳过。失败为三个流程等待超时、
  两个期待 fault 事件的断言和一个期待后端急停的断言；保留现状，尚待专门核对。

未重跑 ROS/原生 C++ 或真机验收；不将历史阶段结果描述为当前全量通过。
现场 .morla_piano 配置/曲谱仍需独立备份，CAN 激活脚本仍需按部署主机补齐。

File: src/robot_description/urdf/nero/xhand_nero_description.urdf (robot description, URDF)
Before this commit: robot xhand_nero, 1282 links, 1281 joints
Joints:
- joint left_hand_index_bend_joint: limit lower=-0.174 upper=0.174 effort=0.4 velocity=14.38 -> lower=-0.08726646259971647 upper=0.29670597283903605 effort=0.4 velocity=14.38
- joint left_hand_index_joint1: limit lower=0 upper=1.919 effort=1.1 velocity=8.63 -> lower=0.0 upper=1.9198621771937625 effort=1.1 velocity=8.63
- joint left_hand_index_joint2: limit lower=0 upper=1.919 effort=0.4 velocity=14.38 -> lower=0.0 upper=1.9198621771937625 effort=0.4 velocity=14.38
- joint left_hand_mid_joint1: limit lower=0 upper=1.919 effort=1.1 velocity=8.63 -> lower=0.0 upper=1.9198621771937625 effort=1.1 velocity=8.63
- joint left_hand_mid_joint2: limit lower=0 upper=1.919 effort=0.4 velocity=14.38 -> lower=0.0 upper=1.9198621771937625 effort=0.4 velocity=14.38
- joint left_hand_pinky_joint1: limit lower=0 upper=1.919 effort=1.1 velocity=8.63 -> lower=0.0 upper=1.9198621771937625 effort=1.1 velocity=8.63
- joint left_hand_pinky_joint2: limit lower=0 upper=1.919 effort=0.4 velocity=14.38 -> lower=0.0 upper=1.9198621771937625 effort=0.4 velocity=14.38
- joint left_hand_ring_joint1: limit lower=0 upper=1.919 effort=1.1 velocity=8.63 -> lower=0.0 upper=1.9198621771937625 effort=1.1 velocity=8.63
- joint left_hand_ring_joint2: limit lower=0 upper=1.919 effort=0.4 velocity=14.38 -> lower=0.0 upper=1.9198621771937625 effort=0.4 velocity=14.38
- joint left_hand_thumb_bend_joint: limit lower=0 upper=1.832 effort=1.1 velocity=8.63 -> lower=0.0 upper=1.5707963267948966 effort=1.1 velocity=8.63
- joint left_hand_thumb_rota_joint1: limit lower=-0.698 upper=1.57 effort=1.1 velocity=8.63 -> lower=-1.0471975511965976 upper=1.5707963267948966 effort=1.1 velocity=8.63
- joint left_hand_thumb_rota_joint2: limit lower=0 upper=1.57 effort=0.4 velocity=14.38 -> lower=0.0 upper=1.5707963267948966 effort=0.4 velocity=14.38
- joint right_hand_index_bend_joint: limit lower=-0.174 upper=0.174 effort=0.4 velocity=14.38 -> lower=-0.08726646259971647 upper=0.29670597283903605 effort=0.4 velocity=14.38
- joint right_hand_index_joint1: limit lower=0 upper=1.919 effort=1.1 velocity=8.63 -> lower=0.0 upper=1.9198621771937625 effort=1.1 velocity=8.63
- joint right_hand_index_joint2: limit lower=0 upper=1.919 effort=0.4 velocity=14.38 -> lower=0.0 upper=1.9198621771937625 effort=0.4 velocity=14.38
- joint right_hand_mid_joint1: limit lower=0 upper=1.919 effort=1.1 velocity=8.63 -> lower=0.0 upper=1.9198621771937625 effort=1.1 velocity=8.63
- joint right_hand_mid_joint2: limit lower=0 upper=1.919 effort=0.4 velocity=14.38 -> lower=0.0 upper=1.9198621771937625 effort=0.4 velocity=14.38
- joint right_hand_pinky_joint1: limit lower=0 upper=1.919 effort=1.1 velocity=8.63 -> lower=0.0 upper=1.9198621771937625 effort=1.1 velocity=8.63
- joint right_hand_pinky_joint2: limit lower=0 upper=1.919 effort=0.4 velocity=14.38 -> lower=0.0 upper=1.9198621771937625 effort=0.4 velocity=14.38
- joint right_hand_ring_joint1: limit lower=0 upper=1.919 effort=1.1 velocity=8.63 -> lower=0.0 upper=1.9198621771937625 effort=1.1 velocity=8.63
- joint right_hand_ring_joint2: limit lower=0 upper=1.919 effort=0.4 velocity=14.38 -> lower=0.0 upper=1.9198621771937625 effort=0.4 velocity=14.38
- joint right_hand_thumb_bend_joint: limit lower=0 upper=1.832 effort=1.1 velocity=8.63 -> lower=0.0 upper=1.5707963267948966 effort=1.1 velocity=8.63
- joint right_hand_thumb_rota_joint1: limit lower=-0.698 upper=1.57 effort=1.1 velocity=8.63 -> lower=-1.0471975511965976 upper=1.5707963267948966 effort=1.1 velocity=8.63
- joint right_hand_thumb_rota_joint2: limit lower=0 upper=1.57 effort=0.4 velocity=14.38 -> lower=0.0 upper=1.5707963267948966 effort=0.4 velocity=14.38

File: src/robot_description/urdf/xhand/xhand_left.urdf (robot description, URDF)
Before this commit: robot xhand_left, 30 links, 29 joints
Joints:
- joint left_hand_index_bend_joint: limit lower=-0.174 upper=0.174 effort=0.4 velocity=14.38 -> lower=-0.08726646259971647 upper=0.29670597283903605 effort=0.4 velocity=14.38
- joint left_hand_index_joint1: limit lower=0 upper=1.919 effort=1.1 velocity=8.63 -> lower=0.0 upper=1.9198621771937625 effort=1.1 velocity=8.63
- joint left_hand_index_joint2: limit lower=0 upper=1.919 effort=0.4 velocity=14.38 -> lower=0.0 upper=1.9198621771937625 effort=0.4 velocity=14.38
- joint left_hand_mid_joint1: limit lower=0 upper=1.919 effort=1.1 velocity=8.63 -> lower=0.0 upper=1.9198621771937625 effort=1.1 velocity=8.63
- joint left_hand_mid_joint2: limit lower=0 upper=1.919 effort=0.4 velocity=14.38 -> lower=0.0 upper=1.9198621771937625 effort=0.4 velocity=14.38
- joint left_hand_pinky_joint1: limit lower=0 upper=1.919 effort=1.1 velocity=8.63 -> lower=0.0 upper=1.9198621771937625 effort=1.1 velocity=8.63
- joint left_hand_pinky_joint2: limit lower=0 upper=1.919 effort=0.4 velocity=14.38 -> lower=0.0 upper=1.9198621771937625 effort=0.4 velocity=14.38
- joint left_hand_ring_joint1: limit lower=0 upper=1.919 effort=1.1 velocity=8.63 -> lower=0.0 upper=1.9198621771937625 effort=1.1 velocity=8.63
- joint left_hand_ring_joint2: limit lower=0 upper=1.919 effort=0.4 velocity=14.38 -> lower=0.0 upper=1.9198621771937625 effort=0.4 velocity=14.38
- joint left_hand_thumb_bend_joint: limit lower=0 upper=1.832 effort=1.1 velocity=8.63 -> lower=0.0 upper=1.5707963267948966 effort=1.1 velocity=8.63
- joint left_hand_thumb_rota_joint1: limit lower=-0.698 upper=1.57 effort=1.1 velocity=8.63 -> lower=-1.0471975511965976 upper=1.5707963267948966 effort=1.1 velocity=8.63
- joint left_hand_thumb_rota_joint2: limit lower=0 upper=1.57 effort=0.4 velocity=14.38 -> lower=0.0 upper=1.5707963267948966 effort=0.4 velocity=14.38

File: src/robot_description/urdf/xhand/xhand_right.urdf (robot description, URDF)
Before this commit: robot xhand_right, 20 links, 19 joints
Joints:
- joint right_hand_index_bend_joint: limit lower=-0.175 upper=0.175 effort=0.4 velocity=14.38 -> lower=-0.08726646259971647 upper=0.29670597283903605 effort=0.4 velocity=14.38
- joint right_hand_index_joint1: limit lower=0 upper=1.92 effort=1.1 velocity=8.63 -> lower=0.0 upper=1.9198621771937625 effort=1.1 velocity=8.63
- joint right_hand_index_joint2: limit lower=0 upper=1.92 effort=0.4 velocity=14.38 -> lower=0.0 upper=1.9198621771937625 effort=0.4 velocity=14.38
- joint right_hand_mid_joint1: limit lower=0 upper=1.92 effort=1.1 velocity=8.63 -> lower=0.0 upper=1.9198621771937625 effort=1.1 velocity=8.63
- joint right_hand_mid_joint2: limit lower=0 upper=1.94 effort=0.4 velocity=14.38 -> lower=0.0 upper=1.9198621771937625 effort=0.4 velocity=14.38
- joint right_hand_pinky_joint1: limit lower=0 upper=1.92 effort=1.1 velocity=8.63 -> lower=0.0 upper=1.9198621771937625 effort=1.1 velocity=8.63
- joint right_hand_pinky_joint2: limit lower=0 upper=1.92 effort=0.4 velocity=14.38 -> lower=0.0 upper=1.9198621771937625 effort=0.4 velocity=14.38
- joint right_hand_ring_joint1: limit lower=0 upper=1.92 effort=1.1 velocity=8.63 -> lower=0.0 upper=1.9198621771937625 effort=1.1 velocity=8.63
- joint right_hand_ring_joint2: limit lower=0 upper=1.92 effort=0.4 velocity=14.38 -> lower=0.0 upper=1.9198621771937625 effort=0.4 velocity=14.38
- joint right_hand_thumb_bend_joint: limit lower=0 upper=1.83 effort=1.1 velocity=8.63 -> lower=0.0 upper=1.5707963267948966 effort=1.1 velocity=8.63
- joint right_hand_thumb_rota_joint1: limit lower=-1.05 upper=1.57 effort=1.1 velocity=8.63 -> lower=-1.0471975511965976 upper=1.5707963267948966 effort=1.1 velocity=8.63
- joint right_hand_thumb_rota_joint2: limit lower=-0.175 upper=1.83 effort=0.4 velocity=14.38 -> lower=0.0 upper=1.5707963267948966 effort=0.4 velocity=14.38
